Commit message: New namespace test

File: linorobot2_description/urdf/controllers/diff_drive.urdf.xacro (robot description, xacro)
@@ -1,8 +1,8 @@
 <robot xmlns:xacro="http://ros.org/wiki/xacro">
-  <xacro:macro name="diff_drive_controller" params="wheel_separation wheel_radius wheel_torque">
+  <xacro:macro name="diff_drive_controller" params="wheel_separation wheel_radius wheel_torque robot_name">
     <gazebo>
       <plugin name="differential_drive_controller" filename="libgazebo_ros_diff_drive.so">
         <ros>
-          <argument>odom:=odom/unfiltered</argument>
+          <argument>odom:=${robot_name}/odom/unfiltered</argument>
         </ros>
         <updateRate>100</updateRate>
@@ -12,9 +12,9 @@
         <wheel_diameter>${wheel_radius * 2}</wheel_diameter>
         <max_wheel_acceleration>1.0</max_wheel_acceleration>
-        <robot_base_frame>base_footprint</robot_base_frame>
+        <robot_base_frame>${robot_name}/base_footprint</robot_base_frame>
         <publish_odom>true</publish_odom>
         <publish_odom_tf>false</publish_odom_tf>
         <publish_wheel_tf>true</publish_wheel_tf>
-        <odometry_frame>odom</odometry_frame>
+        <odometry_frame>${robot_name}/odom</odometry_frame>
       </plugin>
     </gazebo>

File: linorobot2_description/urdf/mech/base.urdf.xacro (robot description, xacro)
@@ -1,5 +1,5 @@
 <?xml version="1.0"?>
 <robot xmlns:xacro="http://ros.org/wiki/xacro">
-  <xacro:macro name="base" params="length width height mass wheel_radius wheel_pos_z">
+  <xacro:macro name="base" params="length width height mass wheel_radius wheel_pos_z robot_name">
     <link name="base_footprint"/>
     <link name="base_link">

File: linorobot2_description/urdf/robots/2wd.urdf.xacro (robot description, xacro)
@@ -1,4 +1,5 @@
 <?xml version="1.0"?>
-<robot name="polybot04" xmlns:xacro="http://ros.org/wiki/xacro">
+<robot name="polybot" xmlns:xacro="http://ros.org/wiki/xacro">
+  <xacro:arg name="robot_name" default="polybot" />
   <xacro:include filename="$(find linorobot2_description)/urdf/2wd_properties.urdf.xacro" />
   <xacro:include filename="$(find linorobot2_description)/urdf/mech/base.urdf.xacro" />
@@ -18,4 +19,5 @@
     wheel_radius="${wheel_radius}"
     wheel_pos_z="${wheel_pos_z}"
+    robot_name="${robot_name}"
 />
   <xacro:layer2/>
@@ -68,4 +70,5 @@
     wheel_radius="${wheel_radius}"
     wheel_torque="${wheel_torque}"
+    robot_name="${robot_name}"
   />
 </robot>
