Commit message: Laser namespace

File: linorobot2_description/urdf/sensors/generic_laser.urdf.xacro (robot description, xacro)
@@ -2,5 +2,5 @@
 <robot xmlns:xacro="http://ros.org/wiki/xacro">
   <xacro:include filename="$(find linorobot2_description)/urdf/sensors/laser.urdf.xacro" />
-  <xacro:macro name="generic_laser" params="*origin">
+  <xacro:macro name="generic_laser" params="*origin robot_name">
     <xacro:laser
       update_rate="10"
@@ -12,4 +12,5 @@
       frame_id="laser"
       topic_name="scan"
+      robot_name="${robot_name}"
     >
       <xacro:insert_block name="origin" />
@@ -26,4 +27,5 @@
       frame_id="base_laser"
       topic_name="base/scan"
+      robot_name="${robot_name}"
     >
       <xacro:insert_block name="origin" />

File: linorobot2_description/urdf/sensors/laser.urdf.xacro (robot description, xacro)
@@ -64,4 +64,5 @@
         <plugin name="${frame_id}_gazebo_ros_head_hokuyo_controller" filename="libgazebo_ros_ray_sensor.so">
           <ros>
+            <namespace>${robot_name}/</namespace>
             <remapping>~/out:=${topic_name}</remapping>
           </ros>
@@ -70,5 +71,5 @@
           <updateRate>${update_rate}</updateRate>
           <topicName>${topic_name}</topicName>
-          <frame_name>${frame_id}</frame_name>
+          <frame_name>${robot_name}/${frame_id}</frame_name>
           <output_type>sensor_msgs/LaserScan</output_type>
         </plugin>

Commit message: Fix test

File: linorobot2_description/urdf/sensors/generic_laser.urdf.xacro (robot description, xacro)
@@ -2,5 +2,5 @@
 <robot xmlns:xacro="http://ros.org/wiki/xacro">
   <xacro:include filename="$(find linorobot2_description)/urdf/sensors/laser.urdf.xacro" />
-  <xacro:macro name="generic_laser" params="*origin robot_name">
+  <xacro:macro name="generic_laser" params="*origin">
     <xacro:laser
       update_rate="10"
@@ -12,5 +12,5 @@
       frame_id="laser"
       topic_name="scan"
-      robot_name="${robot_name}"
+      robot_name="polybot04"
     >
       <xacro:insert_block name="origin" />
@@ -27,5 +27,5 @@
       frame_id="base_laser"
       topic_name="base/scan"
-      robot_name="${robot_name}"
+      robot_name="polybot04"
     >
       <xacro:insert_block name="origin" />
